File: hardware/open-motion-light.kicad_pcb (KiCad board)
At the start: 4 copper layers, 80 x 80 mm, 99 parts, among them J1 TYPE-C-31-M-12, Q1 2N7002, SW1 SW_Push, SW3 SSSS213800, U1 CN3058E, U2 VCNL4020-GS08, U3 MT9284BS6, U4 XYC-PIR224S-S1, U6 CH340X, U7 STM32L051K8Ux

Commit message: Hardware v1.3 first pass
Parts:
- added C25: 100nF, Capacitor_SMD:C_0402_1005Metric, B.Cu at (106.1, 93.5)
- added C26: 100nF, Capacitor_SMD:C_0402_1005Metric, B.Cu at (104.2, 92.1)
- added C27: 10uF, Capacitor_SMD:C_0603_1608Metric, B.Cu at (104.1, 90.9)
- added C28: 100nF, Capacitor_SMD:C_0402_1005Metric, B.Cu at (104.7, 95.1)
- added R17: 4M7, Resistor_SMD:R_0603_1608Metric, B.Cu at (104.7, 96.5)
- added REF**: OSHW-Certification-Mark-Stacked_20x16mm_SilkScreen, OSHWA_Certification_Mark:OSHW-Certification-Mark-Stacked_20x16mm_SilkScreen, B.Cu at (87.8, 128.9)
- added U5: DS8561-30D4, Homebrew:UDFN-4_L1.0-W1.0-P0.65-TL, B.Cu at (104.7, 93.4)
- C14, C21: moved to B.Cu
- C22: value 47uF -> 100nF; footprint Capacitor_SMD:C_1206_3216Metric -> Capacitor_SMD:C_0402_1005Metric; moved to B.Cu
- R21: value 220 -> 2M; footprint Resistor_SMD:R_0402_1005Metric -> Resistor_SMD:R_0603_1608Metric
- R22: value 220 -> 100k
- R40: value 10k -> 1M; footprint Resistor_SMD:R_0603_1608Metric_Pad0.98x0.95mm_HandSolder -> Resistor_SMD:R_0603_1608Metric
- R41: value 2M -> 1M
- R42: value 330k -> 1M; moved to B.Cu
- moved R41 29.5 mm to (86.2, 116.3), turned to 0 degrees
- moved R40 27.9 mm to (88.4, 118.1)
- moved R22 21.7 mm to (79.0, 119.6)
- moved C22 10.6 mm to (116.8, 92.8), turned to 90 degrees
- moved R26 10.1 mm to (118.7, 111.9)
- moved R21 8.66 mm to (85.2, 118.1), turned to 0 degrees
- moved R42 5.20 mm to (110.4, 91.0), turned to 90 degrees
- moved LED2 3.41 mm to (96.7, 87.7)
- moved C14 2.99 mm to (111.7, 90.8)
- moved LED3 2.01 mm to (111.6, 111.9)
- moved C21 1.14 mm to (107.3, 93.5), turned to -90 degrees
Connections:
- C14 pad 1: Net-(U4-VDD) -> Net-(U4-SENS)
- C21 pad 1: Net-(U4-VDD) -> /PIR_3V
- C22 pad 1: GND -> /PIR_3V
- C22 pad 2: Net-(U4-VDD) -> GND
- R21 pad 1: Net-(U6-TXD) -> /SENS_ADJUST_LOW
- R21 pad 2: /USART_RX -> Net-(U4-SENS)
- R22 pad 1: Net-(U6-RXD) -> /PIR_EN
- R22 pad 2: /USART_TX -> /PIR_EN_RAW
- R40 pad 1: VCC -> /SENS_ADJUST_HIGH_1
- R40 pad 2: Net-(U4-VDD) -> Net-(U4-SENS)
- R41 pad 1: Net-(U4-SENS) -> /SENS_ADJUST_HIGH_2
- R41 pad 2: GND -> Net-(U4-SENS)
- R42 pad 1: Net-(U4-VDD) -> Net-(U4-SENS)
- R42 pad 2: Net-(U4-SENS) -> GND
- U4 pad 3: Net-(U4-VDD) -> /PIR_3V
- U6 pad 8: Net-(U6-TXD) -> /USART_RX
- U6 pad 9: Net-(U6-RXD) -> /USART_TX
- U7 pad 22: unconnected-(U7-PA12-Pad22) -> /PIR_EN
- U7 pad 23: unconnected-(U7-PA13-Pad23) -> /SENS_ADJUST_LOW
- U7 pad 24: unconnected-(U7-PA14-Pad24) -> /SENS_ADJUST_HIGH_1
- U7 pad 25: unconnected-(U7-PA15-Pad25) -> /SENS_ADJUST_HIGH_2
Routing:
- net Net-(U4-SENS): track 7.33 -> 59.7 mm, vias 1 -> 3
- net /PIR_EN_RAW: track 0.00 -> 50.2 mm, vias 0 -> 3
- net /USART_RX: track 1.15 -> 48.7 mm, vias 0 -> 4
- net Net-(U6-TXD): track 46.4 -> 0.00 mm, vias 4 -> 0
- net Net-(U4-VDD): track 17.4 -> 0.00 mm
- net /PIR_3V: track 0.00 -> 15.9 mm, vias 0 -> 2
- net Net-(U4-REL): track 8.38 -> 18.8 mm
- net VCC: track 309.0 -> 319.2 mm, vias 20 -> 21
- net /PIR: track 58.2 -> 48.0 mm
- net /SENS_ADJUST_HIGH_1: track 0.00 -> 9.25 mm, vias 0 -> 2
- net /SENS_ADJUST_LOW: track 0.00 -> 8.63 mm, vias 0 -> 2
- net /SENS_ADJUST_HIGH_2: track 0.00 -> 6.50 mm, vias 0 -> 2
- net Net-(LED2-Pad1): track 23.7 -> 29.0 mm
- net Net-(U6-RXD): track 4.97 -> 0.00 mm, vias 2 -> 0
- net /USART_TX: track 43.4 -> 48.2 mm
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Other:
- board text added: "open-motion-light v1.3"
- board text removed: "open-motion-light v1.2"

Commit message: Hardware v1.3 final
Parts:
- removed Q1: 2N7002, Package_TO_SOT_SMD:SOT-23
- removed R10: 100, Resistor_SMD:R_0402_1005Metric
- removed R17: 4M7, Resistor_SMD:R_0603_1608Metric
- removed R22, R38: 100k, Resistor_SMD:R_0402_1005Metric
- removed R32: 22k, Resistor_SMD:R_0402_1005Metric
- removed R33: 330k, Resistor_SMD:R_0603_1608Metric
- removed U5: DS8561-30D4, Homebrew:UDFN-4_L1.0-W1.0-P0.65-TL
- added R43: 82k, Resistor_SMD:R_0402_1005Metric, F.Cu at (79.7, 126.2)
- C1, R3: moved to B.Cu
- C11: value 10uF 28V -> 4.7uF 50V
- C22, C26, C28: moved to F.Cu
- C27: value 10uF -> 100nF; footprint Capacitor_SMD:C_0603_1608Metric -> Capacitor_SMD:C_0402_1005Metric; moved to F.Cu
- F1: value BSMD1206-100-6V -> BSMD1206-075-6V
- L2: value MPL2016S4R7MHT -> 22uH; footprint Homebrew:L0806 -> Inductor_SMD:L_Sunlord_SWPA4030S
- R1: value 24k -> 620; footprint Resistor_SMD:R_0603_1608Metric -> Resistor_SMD:R_0603_1608Metric_Pad0.98x0.95mm_HandSolder
- R2: value 1k5 -> 1k; footprint Resistor_SMD:R_0603_1608Metric -> Resistor_SMD:R_0402_1005Metric
- R25: value 5Ω1 -> 4Ω3
- TH1: footprint Resistor_SMD:R_0402_1005Metric -> Resistor_SMD:R_0603_1608Metric
- U1: value CN3058E -> BQ25170DSGR; footprint Homebrew:SOP-8_3.9x4.9mm_P1.27mm_Thermal -> Homebrew:Texas_DSG0008A_WSON-8-1EP_2x2mm_P0.5mm_EP0.9x1.6mm_ThermalVias
- U3: value MT9284BS6 -> TPS61165DRV; footprint Homebrew:SOT-23-6_L2.9-W1.6-P0.95-LS2.8-BR -> Homebrew:WSON-6-1EP_2x2mm_P0.65mm_EP1x1.6mm_ThermalVias
- moved C22 50.4 mm to (67.6, 103.9), turned to 0 degrees
- moved C1 45.2 mm to (116.6, 87.9)
- moved C28 39.9 mm to (81.4, 127.5), turned to 180 degrees
- moved C26 38.8 mm to (67.6, 104.9)
- moved R3 36.5 mm to (114.1, 95.3)
- moved C27 33.1 mm to (72.8, 101.6), turned to 180 degrees
- moved R13 10.6 mm to (67.2, 93.9)
- moved C21 10.1 mm to (117.4, 92.8), turned to 90 degrees
- moved C25 10.0 mm to (116.1, 92.8), turned to 90 degrees
- moved R25 8.83 mm to (65.1, 104.2), turned to 180 degrees
- moved R2 8.34 mm to (83.7, 122.9), turned to 180 degrees
- moved U3 6.50 mm to (67.2, 102.0), turned to 90 degrees
- moved C24 6.11 mm to (83.9, 128.8)
- moved C11 6.08 mm to (72.7, 103.3), turned to 180 degrees
- moved D8 5.81 mm to (73.2, 99.3)
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Connections:
- net /~{CHRG} renamed /~{PG}
- net /~{DONE} renamed /STAT
- C1 pad 2: +5V -> /PIR_3V
- C22 pad 1: /PIR_3V -> Net-(U3-COMP)
- C26 pad 1: VCC -> Net-(U3-COMP)
- C27 pad 1: VCC -> Net-(D8-K)
- C28 pad 1: /PIR_EN_RAW -> GND
- C28 pad 2: GND -> VCC
- R2 pad 1: Net-(U1-ISET) -> Net-(U1-TS)
- R2 pad 2: Net-(Q1-S) -> /TEMP
- R3 pad 1: Net-(Q1-G) -> VCC
- R3 pad 2: GND -> /PIR_3V
- R34 pad 1: Net-(U3-EN) -> Net-(U3-CTRL)
- R6 pad 2: Net-(U1-~{CHRG}) -> Net-(U1-PG_N)
- R7 pad 2: Net-(U1-~{DONE}) -> Net-(U1-STAT)
- R8 pad 2: Net-(U1-~{DONE}) -> Net-(U1-STAT)
- R9 pad 2: Net-(U1-~{CHRG}) -> Net-(U1-PG_N)
- TH1 pad 1: /TEMP -> Net-(U1-TS)
- U1 pad 1: /TEMP -> +5V
- U1 pad 3: GND -> Net-(U1-TS)
- U1 pad 4: +5V -> GND
- U1 pad 5: VCC -> Net-(U1-STAT)
- U1 pad 6: Net-(U1-~{DONE}) -> Net-(U1-PG_N)
- U1 pad 7: Net-(U1-~{CHRG}) -> Net-(U1-VSET)
- U3 pad 1: Net-(D8-A) -> Net-(U3-FB)
- U3 pad 2: GND -> Net-(U3-COMP)
- U3 pad 3: Net-(U3-FB) -> GND
- U3 pad 4: Net-(U3-EN) -> Net-(D8-A)
- U3 pad 5: Net-(D8-K) -> Net-(U3-CTRL)
- U7 pad 15: unconnected-(U7-PB1-Pad15) -> /TEMP
- U7 pad 22: /PIR_EN -> unconnected-(U7-PA12-Pad22)
- U7 pad 27: /CHARGE_HI_ENABLE -> unconnected-(U7-PB4-Pad27)
Routing:
- net VCC: track 319.2 -> 251.5 mm, vias 21 -> 17
- net GND: track 147.8 -> 93.5 mm, vias 162 -> 160
- net /PIR_EN_RAW: track 50.2 -> 0.00 mm, vias 3 -> 0
- net Net-(U3-CTRL): track 0.00 -> 38.8 mm, vias 0 -> 2
- net Net-(U3-EN): track 25.4 -> 0.00 mm
- net Net-(Q1-G): track 17.9 -> 0.00 mm, vias 2 -> 0
- net Net-(U1-TS): track 0.00 -> 17.8 mm
- net Net-(U3-FB): track 20.2 -> 7.06 mm
- net /TEMP: track 29.0 -> 16.7 mm, vias 4 -> 2
- net Net-(R13-Pad1): track 8.91 -> 2.27 mm
- net Net-(D8-A): track 11.4 -> 5.00 mm, vias 2 -> 0
- net Net-(D8-K): track 12.6 -> 18.1 mm
- net +5V: track 61.5 -> 56.0 mm
- net Net-(U1-STAT): track 0.00 -> 4.83 mm
- net Net-(U1-PG_N): track 0.00 -> 4.59 mm
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